Commit message: 11.11.2025

File: assets/PAROL6.urdf (robot description, URDF)
Before this commit: robot parol6, 8 links, 7 joints
Links:
- link L6: geometry collision mesh filename=package://PAROL6_GUI/assets/VacGrip.STL; visual mesh filename=package://PAROL6_GUI/assets/VacGrip.STL

Commit message: 27.12.2025

File: assets/PAROL6.urdf (robot description, URDF)
Before this commit: robot parol6, 8 links, 7 joints
Links:
- added link tool0
Joints:
- added joint tool0_fixed: type fixed, parent L6, child tool0, origin xyz=0.1 0 -0.04 rpy=0 0 0

Commit message: 08.01.2026

File: assets/PAROL6.urdf (robot description, URDF)
Before this commit: robot parol6, 9 links, 8 joints
Links:
- removed link tool0
Joints:
- removed joint tool0_fixed
